Commit message: more tests

File: lunabot.urdf (robot description, URDF)
Before this commit: robot lunabot, 1 links, 0 joints
Links:
- added link body_link; visual box size=0.505 0.6 0.475
- added link depth_camera_link; visual cylinder length=0.1 radius=0.05
- link base_link: mass 1.0 -> None; geometry 
Joints:
- added joint body_joint: type fixed, parent base_link, child body_link, origin xyz=0 0.3 0.0 rpy=0 0 0
- added joint camera_joint: type fixed, parent base_link, child depth_camera_link, origin xyz=0 0.573 -0.298 rpy=-13.4 0 0

Commit message: more fixes

File: lunabot.urdf (robot description, URDF)
Before this commit: robot lunabot, 3 links, 2 joints
Joints:
- joint camera_joint: origin xyz=0 0.573 -0.298 rpy=-13.4 0 0 -> xyz=0 0.573 -0.298 rpy=-0.23387411976724016330777456297747 0 0
