Commit message: camera enumeration draft

File: urdf/lunabot.urdf (robot description, URDF)
Before this commit: robot lunabot, 3 links, 2 joints
Links:
- added link front_camera; visual cylinder length=0.1 radius=0.05

Commit message: pathfinding tests

File: urdf/lunabot.urdf (robot description, URDF)
Before this commit: robot lunabot, 4 links, 2 joints
Joints:
- joint camera_joint: origin xyz=0 0.573 -0.298 rpy=-0.23387411976724016330777456297747 0 0 -> xyz=0 0.573 -0.298 rpy=-0.52359877559829887307710723054658 0 0
